File: _autosave-powermod.kicad_sch (KiCad schematic)
At the start: 19 parts, among them J1 Conn_02x07_Odd_Even, J2 Conn_02x07_Odd_Even, U2 TPS54260DGQ

Commit message: feat: tps54260
Parts:
- removed D2: PMEG60T30ELR, Diode_SMD:D_SMC-RM10_Universal_Handsoldering, symbol Diode:PMEG60T30ELR
- added D1: B360, Diode_SMD:D_SMC, symbol Diode:B360
Connections:
- net GND: now also D1.2 (A)
- net SW: now also D1.1 (K)
Changed lines of the file:
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@@
+	)
+	(symbol
+		(lib_id "Diode:B360")
+		(at 90.17 26.67 90)
+		(unit 1)
+		(exclude_from_sim no)
+		(in_bom yes)
+		(on_board yes)
+		(dnp no)
+		(fields_autoplaced yes)
+		(property "Reference" "D1"
+			(at 92.71 25.7174 90)
+			(effects
+				(font
+					(size 1.27 1.27)
+				)
+				(justify right)
+			)
+		)
+		(property "Value" "B360"
+			(at 92.71 28.2574 90)
+			(effects
+				(font
+					(size 1.27 1.27)
+				)
+				(justify right)
+			)
+		)
+		(property "Footprint" "Diode_SMD:D_SMC"
+			(at 94.615 26.67 0)
+			(effects
+				(font
+					(size 1.27 1.27)
+				)
+				(hide yes)
+			)
+		)
+		(property "Datasheet" "http://www.jameco.com/Jameco/Products/ProdDS/1538777.pdf"
+			(at 90.17 26.67 0)
+			(effects
+				(font
+					(size 1.27 1.27)
+				)
+				(hide yes)
+			)
+		)
+		(property "Description" "60V 3A Schottky Barrier Rectifier Diode, SMC"
+			(at 90.17 26.67 0)
+			(effects
+				(font
+					(size 1.27 1.27)
+				)
+				(hide yes)
+			)
+		)
+		(pin "1"
+		)
+		(pin "2"
+		)
+		(instances
+			(project ""
+				(path "/4d4b0fcd-2c79-4fc3-b5fa-7a0741601344"
+					(reference "D1")
+					(unit 1)
+				)
+			)
+		)
 	)
 	(symbol
@@
 					(unit 1)
 				)
-			)
-		)
-	)
-	(symbol
-		(lib_id "Diode:PMEG60T30ELR")
-		(at 90.17 26.67 90)
-		(unit 1)
-		(exclude_from_sim no)
-		(in_bom yes)
-		(on_board yes)
-		(dnp no)
-		(fields_autoplaced yes)
-		(property "Reference" "D2"
-			(at 92.71 25.7174 90)
-			(effects
-				(font
-					(size 1.27 1.27)
-				)
-				(justify right)
-			)
-		)
-		(property "Value" "PMEG60T30ELR"
-			(at 92.71 28.2574 90)
-			(effects
-				(font
-					(size 1.27 1.27)
-				)
-				(justify right)
-			)
-		)
-		(property "Footprint" "Diode_SMD:D_SMC-RM10_Universal_Handsoldering"
-			(at 94.615 26.67 0)
-			(effects
-				(font
-					(size 1.27 1.27)
-				)
-				(hide yes)
-			)
-		)
-		(property "Datasheet" "https://assets.nexperia.com/documents/data-sheet/PMEG60T30ELR.pdf"
-			(at 90.17 26.67 0)
-			(effects
-				(font
-					(size 1.27 1.27)
-				)
-				(hide yes)
-			)
-		)
-		(property "Description" "60V, 3A low leakage current Trench MEGA Schottky barrier rectifier, SOD-123W"
-			(at 90.17 26.67 0)
-			(effects
-				(font
-					(size 1.27 1.27)
-				)
-				(hide yes)
-			)
-		)
-		(pin "1"
-		)
-		(pin "2"
-		)
-		(instances
-			(project ""
-				(path "/4d4b0fcd-2c79-4fc3-b5fa-7a0741601344"
-					(reference "D2")
-					(unit 1)
-				)

Commit message: fix: moved and fixed cap footprint
Parts:
- renumbered U2 to U1
Changed lines of the file:
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@@
 		(dnp no)
 		(fields_autoplaced yes)
-		(property "Reference" "U2"
+		(property "Reference" "U1"
 			(at 63.5 27.94 0)
 			(effects
@@
 			(project "powermod"
 				(path "/4d4b0fcd-2c79-4fc3-b5fa-7a0741601344"
-					(reference "U2")
+					(reference "U1")
 					(unit 1)
 				)

Commit message: feat: powermod-tps54260-1.0-1 production files
Parts:
- C2: footprint Capacitor_SMD:C_0402_1005Metric -> Capacitor_SMD:C_0603_1608Metric
Changed lines of the file:
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@@
 			)
 		)
-		(property "Footprint" "Capacitor_SMD:C_0402_1005Metric"
+		(property "Footprint" "Capacitor_SMD:C_0603_1608Metric"
 			(at 33.9852 38.1 0)
 			(effects

Commit message: feat: changes
Parts:
- removed C2: 2.2uF, Capacitor_SMD:C_0603_1608Metric, symbol Device:C
- C1: value 2.2uF -> 22uF 2201010609TR; footprint Capacitor_SMD:C_0603_1608Metric -> Capacitor_SMD:C_Elec_6.3x7.7
- L1: value 10uH -> 15uH
- R2: value 52.5K -> 59K
- R3: value 10K -> 11K

Commit message: fix: now delivers 1.5 amps
Parts:
- C5: value 100pF -> 100uF
- L1: value 15uH -> 10uH
- R2: value 59K -> 52K
- R7: value 237K -> 43K
- R8: value 29K -> 9K
Changed lines of the file:
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@@
 			)
 		)
-		(property "Value" "15uH"
+		(property "Value" "10uH"
 			(at 96.52 33.0454 90)
 			(effects
@@
 			)
 		)
-		(property "Value" "100pF"
+		(property "Value" "100uF"
 			(at 95.25 41.91 0)
 			(effects
@@
 			)
 		)
-		(property "Value" "59K"
+		(property "Value" "52K"
 			(at 119.38 44.45 0)
 			(effects
@@
 			)
 		)
-		(property "Value" "237K"
+		(property "Value" "43K"
 			(at 40.64 54.61 0)
 			(effects
@@
 			)
 		)
-		(property "Value" "29K"
+		(property "Value" "9K"
 			(at 50.8 59.69 0)
 			(effects
